File: hardware/SKnob.sch (KiCad schematic (older format))
At the start: 3 parts, among them U1 STM32WLE5JCI6

Commit message: antena section
Parts:
- added C? (x10): C, symbol Device:C
- added L? (x5): L, symbol Device:L
Connections:
- wire segments 38 -> 76

Commit message: rf network
Parts:
- removed U1: STM32WLE5JCI6, SKnob:STM32WLE5JCI6, symbol STM32WLE5JCI6:STM32WLE5JCI6
- added C11, C12, C13: C, Capacitor_SMD:C_0402_1005Metric, symbol Device:C
- added L6: L, Inductor_SMD:L_0402_1005Metric, symbol Device:L
- added U1: STM32WLE5JCI6, SKnob:STM32WLE5JCI6, symbol SKnob:STM32WLE5JCI6
- added U2: BGS12SN6, Package_BGA:Texas_DSBGA-6_0.9x1.4mm_Layout2x3_P0.5mm, symbol SKnob:BGS12SN6
- C1, C10, C2, C3, C4, C5, C6, C7, C8, C9: renamed from C?; footprint (none) -> Capacitor_SMD:C_0402_1005Metric
- L1, L2, L3, L4, L5: renamed from L?; footprint (none) -> Inductor_SMD:L_0402_1005Metric
Connections:
- net labels added: RFI_N, RFI_P, RFO_LP
- wire segments 76 -> 86
- no-connect marks 0 -> 1
Changed lines of the file:
@@
 Comment4 ""
 $EndDescr
-$Comp
-L STM32WLE5JCI6:STM32WLE5JCI6 U1
-U 1 1 5EC5E3A0
-P 3950 5300
-F 0 "U1" H 5250 5787 60  0000 C CNN
-F 1 "STM32WLE5JCI6" H 5250 5681 60  0000 C CNN
-F 2 "SKnob:STM32WLE5JCI6" H 5250 5640 60  0001 C CNN
-F 3 "" H 3950 5300 60  0000 C CNN
-	1    3950 5300
-	1    0    0    -1
-$EndComp
-$Comp
-L STM32WLE5JCI6:STM32WLE5JCI6 U1
-U 2 1 5EC5F9D6
-P 11600 5750
-F 0 "U1" H 12900 6137 60  0000 C CNN
-F 1 "STM32WLE5JCI6" H 12900 6031 60  0000 C CNN
-F 2 "SKnob:STM32WLE5JCI6" H 12900 6090 60  0001 C CNN
-F 3 "" H 11600 5750 60  0000 C CNN
-	2    11600 5750
-	1    0    0    -1
-$EndComp
 Text Label 6850 5700 2    50   ~ 0
 PA0
@@
 L Device:Antenna_Chip AE1
 U 1 1 5EC5B94F
-P 10150 2250
-F 0 "AE1" H 10330 2377 50  0000 L CNN
-F 1 "Antenna_Chip" H 10330 2286 50  0000 L CNN
-F 2 "" H 10050 2425 50  0001 C CNN
-F 3 "~" H 10050 2425 50  0001 C CNN
-	1    10150 2250
-	1    0    0    -1
-$EndComp
-$Comp
-L Device:L L?
+P 12550 2050
+F 0 "AE1" H 12730 2177 50  0000 L CNN
+F 1 "Antenna_Chip" H 12730 2086 50  0000 L CNN
+F 2 "" H 12450 2225 50  0001 C CNN
+F 3 "~" H 12450 2225 50  0001 C CNN
+	1    12550 2050
+	1    0    0    -1
+$EndComp
+$Comp
+L Device:L L2
 U 1 1 5ECC217D
 P 5500 1850
-F 0 "L?" V 5690 1850 50  0000 C CNN
+F 0 "L2" V 5690 1850 50  0000 C CNN
 F 1 "L" V 5599 1850 50  0000 C CNN
-F 2 "" H 5500 1850 50  0001 C CNN
+F 2 "Inductor_SMD:L_0402_1005Metric" H 5500 1850 50  0001 C CNN
 F 3 "~" H 5500 1850 50  0001 C CNN
 	1    5500 1850
@@
 $EndComp
 $Comp
-L Device:L L?
+L Device:L L3
 U 1 1 5ECC2B95
 P 5900 1100
-F 0 "L?" H 5953 1146 50  0000 L CNN
+F 0 "L3" H 5953 1146 50  0000 L CNN
 F 1 "L" H 5953 1055 50  0000 L CNN
-F 2 "" H 5900 1100 50  0001 C CNN
+F 2 "Inductor_SMD:L_0402_1005Metric" H 5900 1100 50  0001 C CNN
 F 3 "~" H 5900 1100 50  0001 C CNN
 	1    5900 1100
@@
 $EndComp
 $Comp
-L Device:L L?
+L Device:L L4
 U 1 1 5ECC315A
 P 6750 1850
-F 0 "L?" V 6940 1850 50  0000 C CNN
+F 0 "L4" V 6940 1850 50  0000 C CNN
 F 1 "L" V 6849 1850 50  0000 C CNN
-F 2 "" H 6750 1850 50  0001 C CNN
+F 2 "Inductor_SMD:L_0402_1005Metric" H 6750 1850 50  0001 C CNN
 F 3 "~" H 6750 1850 50  0001 C CNN
 	1    6750 1850
@@
 $EndComp
 $Comp
-L Device:C C?
+L Device:C C7
 U 1 1 5ECC3643
 P 6750 1450
-F 0 "C?" V 6498 1450 50  0000 C CNN
+F 0 "C7" V 6498 1450 50  0000 C CNN
 F 1 "C" V 6589 1450 50  0000 C CNN
-F 2 "" H 6788 1300 50  0001 C CNN
+F 2 "Capacitor_SMD:C_0402_1005Metric" H 6788 1300 50  0001 C CNN
 F 3 "~" H 6750 1450 50  0001 C CNN
 	1    6750 1450
@@
 $EndComp
 $Comp
-L Device:C C?
+L Device:C C6
 U 1 1 5ECC399D
 P 6450 2200
-F 0 "C?" H 6565 2246 50  0000 L CNN
+F 0 "C6" H 6565 2246 50  0000 L CNN
 F 1 "C" H 6565 2155 50  0000 L CNN
-F 2 "" H 6488 2050 50  0001 C CNN
+F 2 "Capacitor_SMD:C_0402_1005Metric" H 6488 2050 50  0001 C CNN
 F 3 "~" H 6450 2200 50  0001 C CNN
 	1    6450 2200
@@
 $EndComp
 $Comp
-L Device:C C?
+L Device:C C8
 U 1 1 5ECC3DD4
 P 7050 2200
-F 0 "C?" H 7165 2246 50  0000 L CNN
+F 0 "C8" H 7165 2246 50  0000 L CNN
 F 1 "C" H 7165 2155 50  0000 L CNN
-F 2 "" H 7088 2050 50  0001 C CNN
+F 2 "Capacitor_SMD:C_0402_1005Metric" H 7088 2050 50  0001 C CNN
 F 3 "~" H 7050 2200 50  0001 C CNN
 	1    7050 2200
@@
 $EndComp
 $Comp
-L Device:C C?
+L Device:C C9
 U 1 1 5ECC4152
 P 7350 1850
-F 0 "C?" V 7098 1850 50  0000 C CNN
+F 0 "C9" V 7098 1850 50  0000 C CNN
 F 1 "C" V 7189 1850 50  0000 C CNN
-F 2 "" H 7388 1700 50  0001 C CNN
+F 2 "Capacitor_SMD:C_0402_1005Metric" H 7388 1700 50  0001 C CNN
 F 3 "~" H 7350 1850 50  0001 C CNN
 	1    7350 1850
@@
 $EndComp
 $Comp
-L Device:L L?
+L Device:L L5
 U 1 1 5ECC43C8
 P 7950 1850
-F 0 "L?" V 8140 1850 50  0000 C CNN
+F 0 "L5" V 8140 1850 50  0000 C CNN
 F 1 "L" V 8049 1850 50  0000 C CNN
-F 2 "" H 7950 1850 50  0001 C CNN
+F 2 "Inductor_SMD:L_0402_1005Metric" H 7950 1850 50  0001 C CNN
 F 3 "~" H 7950 1850 50  0001 C CNN
 	1    7950 1850
@@
 $EndComp
 $Comp
-L Device:C C?
+L Device:C C10
 U 1 1 5ECC4768
 P 8250 2200
-F 0 "C?" H 8365 2246 50  0000 L CNN
+F 0 "C10" H 8365 2246 50  0000 L CNN
 F 1 "C" H 8365 2155 50  0000 L CNN
-F 2 "" H 8288 2050 50  0001 C CNN
+F 2 "Capacitor_SMD:C_0402_1005Metric" H 8288 2050 50  0001 C CNN
 F 3 "~" H 8250 2200 50  0001 C CNN
 	1    8250 2200
@@
 $EndComp
 $Comp
-L Device:C C?
+L Device:C C3
 U 1 1 5ECC4A3A
 P 5450 1100
-F 0 "C?" H 5565 1146 50  0000 L CNN
+F 0 "C3" H 5565 1146 50  0000 L CNN
 F 1 "C" H 5565 1055 50  0000 L CNN
-F 2 "" H 5488 950 50  0001 C CNN
+F 2 "Capacitor_SMD:C_0402_1005Metric" H 5488 950 50  0001 C CNN
 F 3 "~" H 5450 1100 50  0001 C CNN
 	1    5450 1100
@@
 $EndComp
 $Comp
-L Device:C C?
+L Device:C C1
 U 1 1 5ECC4DB8
 P 5000 1100
-F 0 "C?" H 5115 1146 50  0000 L CNN
+F 0 "C1" H 5115 1146 50  0000 L CNN
 F 1 "C" H 5115 1055 50  0000 L CNN
-F 2 "" H 5038 950 50  0001 C CNN
+F 2 "Capacitor_SMD:C_0402_1005Metric" H 5038 950 50  0001 C CNN
 F 3 "~" H 5000 1100 50  0001 C CNN
 	1    5000 1100
@@
 $EndComp
 $Comp
-L Device:C C?
+L Device:C C5
 U 1 1 5ECC51E2
 P 6000 3000
-F 0 "C?" H 6115 3046 50  0000 L CNN
+F 0 "C5" H 6115 3046 50  0000 L CNN
 F 1 "C" H 6115 2955 50  0000 L CNN
-F 2 "" H 6038 2850 50  0001 C CNN
+F 2 "Capacitor_SMD:C_0402_1005Metric" H 6038 2850 50  0001 C CNN
 F 3 "~" H 6000 3000 50  0001 C CNN
 	1    6000 3000
@@
 $EndComp
 $Comp
-L Device:C C?
+L Device:C C4
 U 1 1 5ECC5686
 P 5500 2650
-F 0 "C?" V 5248 2650 50  0000 C CNN
+F 0 "C4" V 5248 2650 50  0000 C CNN
 F 1 "C" V 5339 2650 50  0000 C CNN
-F 2 "" H 5538 2500 50  0001 C CNN
+F 2 "Capacitor_SMD:C_0402_1005Metric" H 5538 2500 50  0001 C CNN
 F 3 "~" H 5500 2650 50  0001 C CNN
 	1    5500 2650
@@
 $EndComp
 $Comp
-L Device:L L?
+L Device:L L1
 U 1 1 5ECC5ED8
 P 5100 3000
-F 0 "L?" H 5153 3046 50  0000 L CNN
+F 0 "L1" H 5153 3046 50  0000 L CNN
 F 1 "L" H 5153 2955 50  0000 L CNN
-F 2 "" H 5100 3000 50  0001 C CNN
+F 2 "Inductor_SMD:L_0402_1005Metric" H 5100 3000 50  0001 C CNN
 F 3 "~" H 5100 3000 50  0001 C CNN
 	1    5100 3000
@@
 $EndComp
 $Comp
-L Device:C C?
+L Device:C C2
 U 1 1 5ECC7D54
 P 5100 3450
-F 0 "C?" H 5215 3496 50  0000 L CNN
+F 0 "C2" H 5215 3496 50  0000 L CNN
 F 1 "C" H 5215 3405 50  0000 L CNN
-F 2 "" H 5138 3300 50  0001 C CNN
+F 2 "Capacitor_SMD:C_0402_1005Metric" H 5138 3300 50  0001 C CNN
 F 3 "~" H 5100 3450 50  0001 C CNN
 	1    5100 3450
@@
 	8250 1850 8900 1850
 Wire Wire Line
-	8900 2650 8900 2350
-Wire Wire Line
-	8900 2350 9250 2350
+	8900 2650 8900 2250
+Wire Wire Line
+	8900 2250 9250 2250
 Wire Wire Line
 	6000 2850 6000 2650
@@
 Wire Wire Line
 	5450 850  5000 850
+Text Label 6900 5500 2    50   ~ 0
+RFO_LP
+Wire Wire Line
+	6900 5500 6550 5500
+Text Label 3650 5600 0    50   ~ 0
+RFI_P
+Text Label 3650 5500 0    50   ~ 0
+RFI_N
+Wire Wire Line
+	3650 5500 3950 5500
+Wire Wire Line
+	3650 5600 3950 5600
+Text Label 4350 2650 0    50   ~ 0
+RFI_P
+Text Label 4350 3250 0    50   ~ 0
+RFI_N
+Text Label 4350 1850 0    50   ~ 0
+RFO_LP
+$Comp
+L SKnob:BGS12SN6 U2
+U 1 1 5ECE0163
+P 9350 2150
+F 0 "U2" H 9675 2681 50  0000 C CNN
+F 1 "BGS12SN6" H 9675 2590 50  0000 C CNN
+F 2 "Package_BGA:Texas_DSBGA-6_0.9x1.4mm_Layout2x3_P0.5mm" H 9350 2150 50  0001 C CNN
+F 3 "" H 9350 2150 50  0001 C CNN
+	1    9350 2150
+	1    0    0    -1
+$EndComp
+$Comp
+L SKnob:STM32WLE5JCI6 U1
+U 1 1 5ECE49FF
+P 3950 5300
+F 0 "U1" H 5250 5787 60  0000 C CNN
+F 1 "STM32WLE5JCI6" H 5250 5681 60  0000 C CNN
+F 2 "SKnob:STM32WLE5JCI6" H 5250 5640 60  0001 C CNN
+F 3 "" H 3950 5300 60  0000 C CNN
+	1    3950 5300
+	1    0    0    -1
+$EndComp
+$Comp
+L SKnob:STM32WLE5JCI6 U1
+U 2 1 5ECE6D2C
+P 10450 5900
+F 0 "U1" H 11750 6287 60  0000 C CNN
+F 1 "STM32WLE5JCI6" H 11750 6181 60  0000 C CNN
+F 2 "SKnob:STM32WLE5JCI6" H 11750 6240 60  0001 C CNN
+F 3 "" H 10450 5900 60  0000 C CNN
+	2    10450 5900
+	1    0    0    -1
+$EndComp
+$Comp
+L Device:C C11
+U 1 1 5ECE93AF
+P 10500 2150
+F 0 "C11" V 10248 2150 50  0000 C CNN
+F 1 "C" V 10339 2150 50  0000 C CNN
+F 2 "Capacitor_SMD:C_0402_1005Metric" H 10538 2000 50  0001 C CNN
+F 3 "~" H 10500 2150 50  0001 C CNN
+	1    10500 2150
+	0    1    1    0
+$EndComp
+$Comp
+L Device:L L6
+U 1 1 5ECED777
+P 11500 2150
+F 0 "L6" V 11690 2150 50  0000 C CNN
+F 1 "L" V 11599 2150 50  0000 C CNN
+F 2 "Inductor_SMD:L_0402_1005Metric" H 11500 2150 50  0001 C CNN
+F 3 "~" H 11500 2150 50  0001 C CNN
+	1    11500 2150
+	0    -1   -1   0
+$EndComp
+$Comp
+L Device:C C12
+U 1 1 5ECED77D
+P 11200 2500
+F 0 "C12" H 11315 2546 50  0000 L CNN
+F 1 "C" H 11315 2455 50  0000 L CNN
+F 2 "Capacitor_SMD:C_0402_1005Metric" H 11238 2350 50  0001 C CNN
+F 3 "~" H 11200 2500 50  0001 C CNN
+	1    11200 2500
+	1    0    0    -1
+$EndComp
+$Comp
+L Device:C C13
+U 1 1 5ECED783
+P 11800 2500
+F 0 "C13" H 11915 2546 50  0000 L CNN
+F 1 "C" H 11915 2455 50  0000 L CNN
+F 2 "Capacitor_SMD:C_0402_1005Metric" H 11838 2350 50  0001 C CNN
+F 3 "~" H 11800 2500 50  0001 C CNN
+	1    11800 2500
+	1    0    0    -1
+$EndComp
+$Comp
+L power:GND #PWR?
+U 1 1 5ECED78A
+P 11800 2650
+F 0 "#PWR?" H 11800 2400 50  0001 C CNN
+F 1 "GND" H 11805 2477 50  0000 C CNN
+F 2 "" H 11800 2650 50  0001 C CNN
+F 3 "" H 11800 2650 50  0001 C CNN
+	1    11800 2650
+	1    0    0    -1
+$EndComp
+$Comp
+L power:GND #PWR?
+U 1 1 5ECED790
+P 11200 2650
+F 0 "#PWR?" H 11200 2400 50  0001 C CNN
+F 1 "GND" H 11205 2477 50  0000 C CNN
+F 2 "" H 11200 2650 50  0001 C CNN
+F 3 "" H 11200 2650 50  0001 C CNN
+	1    11200 2650
+	1    0    0    -1
+$EndComp
+Wire Wire Line
+	11200 2350 11200 2150
+Connection ~ 11200 2150
+Wire Wire Line
+	11800 2350 11800 2150
+Connection ~ 11800 2150
+Wire Wire Line
+	10650 2150 11200 2150
+Wire Wire Line
+	11650 2150 11800 2150
+Wire Wire Line
+	11200 2150 11350 2150
+Wire Wire Line
+	10350 2150 10100 2150
+Wire Wire Line
+	11800 2150 12450 2150
+NoConn ~ 12650 2150
 $EndSCHEMATC

Commit message: stm32wb chip selection
Parts:
- removed AE1: Antenna_Chip, symbol Device:Antenna_Chip
- removed C11, C12, C13: C, Capacitor_SMD:C_0402_1005Metric, symbol Device:C
- removed L4, L5, L6: L, Inductor_SMD:L_0402_1005Metric, symbol Device:L
- removed U1: STM32WLE5JCI6, SKnob:STM32WLE5JCI6, symbol SKnob:STM32WLE5JCI6
- removed U2: BGS12SN6, Package_BGA:Texas_DSBGA-6_0.9x1.4mm_Layout2x3_P0.5mm, symbol SKnob:BGS12SN6
- added ANT1: W3008, SKnob:W3008, symbol SKnob:W3008
- added J1: USB_B_Micro, Connector_USB:USB_Micro-B_Molex-105133-0001, symbol Connector:USB_B_Micro
- added U1: STM32WB55Cx, SKnob:STM32WB55Cx, symbol SKnob:STM32WB55Cx
- C1, C2, C3, C4, C7, C8: value C -> 100nF
- C5, C6: value C -> 100pF
- L1, L2: footprint Inductor_SMD:L_0402_1005Metric -> Inductor_SMD:L_0603_1608Metric
Connections:
- net labels added: +5V
- net labels removed: PA0, PA1, PA10, PA11, PA12, PA13, PA14, PA15, PA2, PA3, PA4, PA5, PA6, PA7, PA8, PA9, PB1, PB10, PB11, PB12, PB13, PB14, PB15, PB2, PB3, PB4, PB5, PB6, PB7, PB8, PB9, PC0, PC1, PC2, PC3, PC4, PC5, PC6, RFI_N, RFI_P, RFO_LP
- wire segments 86 -> 48
- no-connect marks 1 -> 0
Other:
- note added: "TODO: pin check 22\npin 30\nsymbol position of pin 30\n\n\n"

Commit message: preliminary routing
Parts:
- removed unit 2 of U1
- added C11, C12, C14, C21, C22, C24: 100nF, Capacitor_SMD:C_0402_1005Metric, symbol Device:C
- added C13, C15, C20, C23, C25, C26: 4.7uF, Capacitor_SMD:C_0805_2012Metric, symbol Device:C
- added C16, C17, C18, C19: C, Capacitor_SMD:C_0402_1005Metric, symbol Device:C
- added D1: D, Diode_SMD:D_0603_1608Metric, symbol Device:D
- added D2: TPD4S012DRYR, SKnob:TPD4S012DRYR, symbol SKnob:TPD4S012DRYR
- added J2, J3: Conn_01x02, Connector_PinHeader_1.00mm:PinHeader_1x02_P1.00mm_Vertical, symbol Connector:Conn_01x02_Female
- added L4: 600R @ 100MHz, Inductor_SMD:L_0402_1005Metric, symbol Device:L
- added R1, R2: R, Resistor_SMD:R_0402_1005Metric, symbol Device:R
- added R3: 10K, Resistor_SMD:R_0402_1005Metric, symbol Device:R
- added R4: 10k, Resistor_SMD:R_0402_1005Metric, symbol Device:R
- added SW1: SW_Push, Button_Switch_SMD:SW_SPST_B3U-3000P, symbol Switch:SW_Push
- added Y1, Y2: 32MHz, Crystal:Crystal_SMD_2016-4Pin_2.0x1.6mm, symbol Device:Crystal_GND24
- BT1: value Battery_Cell -> BR1225; Capacity (none) -> 50mA
- C1: value 100nF -> C
- C10: value C -> 0.3pF
- C6: value 100pF -> 4.7uF; footprint Capacitor_SMD:C_0402_1005Metric -> Capacitor_SMD:C_0805_2012Metric
- C9: value C -> 0.8pF
- L1, L2: value L -> 600R @ 100MHz
- L3: value L -> 2.7nF
Connections:
- net labels added: BOOT, ID, OSC32_IN, OSC32_OUT, OSC_IN, OSC_OUT, RF1, RF1_ANT, USB_N, USB_P
- wire segments 48 -> 131
- no-connect marks 0 -> 1
Other:
- note added: "TODO: Calculate 50 Ohm trace\n"
- note added: "TODO: Change ESD\n"
- note removed: "TODO: pin check 22\npin 30\nsymbol position of pin 30\n\n\n"
- moved on the sheet: ANT1, BT1, C10, C2, C3, C4, C5, C7, C8, C9, J1, L1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

Commit message: added accel
Parts:
- added C27: 100nF, Capacitor_SMD:C_0402_1005Metric, symbol Device:C
- added U2: LIS2DE12TR, SKnob:LIS2DE12TR, symbol SKnob:LIS2DE12TR
Connections:
- net +BATT: now also C27.1, U2.10 (VDD_IO), U2.9 (VDD)
- net GND: now also C27.2, U2.6 (GND), U2.7 (GND), U2.8 (GND)
- net I2C1_SCL: now reaches U1.5 (PB8)
- net I2C1_SCL: now also U2.1 (SCL/SPC)
- net I2C1_SDA: now reaches U1.6 (PB9)
- net I2C1_SDA: now also U2.4 (SDA/SDI/SDO)
Other:
- note removed: "TODO: Calculate 50 Ohm trace\n"
- moved on the sheet: ANT1, BT1, C1, C10, C11, C12, C13, C14, C15, C16, C17, C18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

Commit message: update hardware to include test points in the back and commit auto generated firmware project files
Parts:
- removed D2: TPD4S012DRYR, SKnob:TPD4S012DRYR, symbol SKnob:TPD4S012DRYR
- added R5: 0, SKnob:R_0402_1005Metric_DNP, symbol Device:R
- added T1, T2: LA_LOGO, SKnob:LA_LOGO, symbol SKnob:LA_LOGO
- added TP1, TP10, TP11, TP12, TP13, TP14, TP15, TP16, TP17, TP2, TP3, TP4, TP5, TP6, TP7, TP8, TP9: TestPoint, SKnob:TestPoint_Pad_D1.0mm, symbol Connector:TestPoint
- added U3: USBLC6-2P6, Package_TO_SOT_SMD:SOT-666, symbol Power_Protection:USBLC6-2P6
- C16, C17, C18, C19: value C -> 4.3pF
- C23: value 4.7uF -> 100nF; footprint Capacitor_SMD:C_0805_2012Metric -> Capacitor_SMD:C_0402_1005Metric
- D1: value D -> 1N4148; footprint Diode_SMD:D_0603_1608Metric -> Diode_SMD:D_0402_1005Metric; digikey# (none) -> 1N4148WL2-TPMSCT-ND; manf (none) -> Micro Commercial Co; manf# (none) -> 1N4148WL2-TP
- J2, J3: footprint Connector_PinHeader_1.00mm:PinHeader_1x02_P1.00mm_Vertical -> Connector_PinHeader_2.00mm:PinHeader_1x02_P2.00mm_Vertical
- L4: value 600R @ 100MHz -> 10uH; footprint Inductor_SMD:L_0402_1005Metric -> Inductor_SMD:L_0603_1608Metric; digikey# (none) -> 587-1720-1-ND; manf (none) -> Taiyo Yuden; manf# (none) -> CBMF1608T100K
- R2: value R -> 10k
- R3: footprint Resistor_SMD:R_0402_1005Metric -> SKnob:R_0402_1005Metric_DNP
- Y2: value 32MHz -> 32.768kHz
Connections:
- net +5V: now also U3.5 (VBUS)
- net +BATT: now also U1.15 (PA6), U2.2 (CS), R5.1; no longer C23.1
- net GND: now also D1.1 (K), U2.5 (RES), U3.2 (GND); no longer SW1.2
- net I2C1_SCL: now also TP2.1
- net I2C1_SDA: now also TP3.1
- net ID: now also U3.1 (I/O1)
- net USB_N: now also U3.4 (I/O2)
- net USB_P: now also U3.3 (I/O2)
- net ACC_INT1: now reaches U1.11 (PA2)
- net ACC_INT1: now also U2.12 (INT1)
- net ACC_INT2: now reaches U1.12 (PA3)
- net ACC_INT2: now also U2.11 (INT2)
- net RCC_MCO: now reaches U1.17 (PA8)
- net RCC_MCO: now also TP1.1
- net USART1_TX: now reaches U1.18 (PA9)
- net USART1_TX: now also TP4.1
- net PB2: now reaches U1.19 (PB2)
- net PB2: now also TP8.1
- net VDDRF: now reaches C5.1, C7.1, L2.1, U1.23 (VDDRF)
- net PB0: now reaches U1.28 (PB0)
- net PB0: now also TP6.1
- net PB1: now reaches U1.29 (PB1)
- net PB1: now also TP7.1
- net at U1.31 (VFBSMPS): now also L4.1, R5.2
- net at U1.33 (VLXSMPS): now also C13.1, L4.2
- net USART1_RX: now reaches U1.36 (PA10)
- net USART1_RX: now also TP5.1
- net JTMS-SWDIO: now reaches U1.39 (PA13)
- net JTMS-SWDIO: now also TP14.1
- net JTCK-SWCLK: now reaches U1.41 (PA14)
- net JTCK-SWCLK: now also TP15.1
- net JTDI: now reaches U1.42 (PA15)
- net JTDI: now also TP16.1
- net PB3_JTDO-SWO: now reaches U1.43 (PB3)
- net PB3_JTDO-SWO: now also TP9.1
- net PB4_JTRST: now reaches U1.44 (PB4)
- net PB4_JTRST: now also TP10.1
- net PB5: now reaches U1.45 (PB5)
- net PB5: now also TP11.1
- net PB6: now reaches U1.46 (PB6)
- net PB6: now also TP12.1
- net PB7: now reaches U1.47 (PB7)
- net PB7: now also TP13.1
- net RST_N: now reaches R2.2, U1.7 (NRST)
- net RST_N: now also C23.1, SW1.1; no longer D1.2 (A)
- net VDDA: now reaches C4.1, L1.1, U1.8 (VDDA)
- net WKUP1: now reaches U1.9 (PA0)
- net WKUP1: now also TP17.1
- new net: D1.2 (A), SW1.2
- no-connect marks 1 -> 9
Other:
- note added: "Analog ADC"
- note removed: "TODO: Change ESD\n"
- moved on the sheet: BT1, C14, C15, C25, C26, D1, L4, R2, SW1

Commit message: finishing touches
Parts:
- removed C10: 0.3pF, Capacitor_SMD:C_0402_1005Metric, symbol Device:C
- removed C9: 0.8pF, Capacitor_SMD:C_0402_1005Metric, symbol Device:C
- removed L3: 2.7nF, Inductor_SMD:L_0402_1005Metric, symbol Device:L
- added BATT?1: BR1225, SKnob:BR1225, symbol SKnob:BR1225
- added FLT1: MLPF-WB55-01E3, SKnob:MLPF-WB55-01E3, symbol SKnob:MLPF-WB55-01E3
- added TP18, TP19: TestPoint, SKnob:TestPoint_Pad_D1.0mm, symbol Connector:TestPoint
- ANT1: Info (none) -> 2.4GHz Bluetooth Chip RF Antenna 2.4GHz ~ 2.483GHz 1.7dBi S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
- BT1: value BR1225 -> BK-885-TR; Capacity 50mA -> (none); Info (none) -> Battery Retainer Coin, 12.0mm 1 Cell SMD (SMT) Tab; digikey# (none) -> BK-885-CT-ND; manf (none) -> MPD (Memory Protection Devices); manf# (none) -> BK-885-TR
- C16, C17, C18, C19: value 4.3pF -> 15pF
- D1: Info (none) -> Diode Standard 100V 150mA Surface Mount DFN1006-2
- L4: Info (none) -> 10µH Unshielded Wirewound Inductor 380mA 468mOhm Max 0603 (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
- U1: Info (none) -> IC RF TxRx + MCU 802.15.4, Bluetooth Bluetooth v5.0 2.405GH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; digikey# (none) -> 497-18489-ND; manf (none) -> STMicroelectronics; manf# (none) -> STM32WB55CGU6
- U2: Info (none) -> Accelerometer X, Y, Z Axis ±2g, 4g, 8g, 16g 0.5Hz ~ 2.69kHz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; digikey# 497-15997-1-ND -> 497-15997-1-ND; manf ST MICROELECTRONICS -> STMicroelectronics
- U3: Info (none) -> 17V Clamp 5A (8/20µs) Ipp Tvs Diode Surface Mount SOT-666; digikey# (none) -> 497-5026-1-ND; manf (none) -> STMicroelectronics; manf# (none) -> USBLC6-2P6
- Y1: Info (none) -> 32MHz ±10ppm Crystal 10pF 60 Ohms 4-SMD, No Lead; digikey# (none) -> 490-18335-1-ND; manf (none) -> Murata Electronics; manf# (none) -> XRCGB32M000F1H02R0
Connections:
- net ACC_INT1: now also U1.13 (PA4); no longer U1.11 (PA2)
- net ACC_INT2: now also U1.14 (PA5); no longer U1.12 (PA3)
- net GND: now also FLT1.2 (GND), FLT1.4 (GND), FLT1.5 (GND), FLT1.6 (GND)
- net RF1: now also FLT1.1 (IN)
- net RF1_ANT: now also FLT1.3 (OUT)
- new net LPUART1_RX: TP19.1, U1.12 (PA3)
- new net LPUART1_TX: TP18.1, U1.11 (PA2)
- no-connect marks 9 -> 7
Other:
- note added: "3-AXIS ACCEL"
- note added: "BATTERY"
- note added: "BOOT"
- note added: "MCU-BLE"
- note added: "OSC"
- note added: "POWER IN"
- note added: "USB"
- moved on the sheet: ANT1, BT1, C1, C11, C12, C13, C14, C15, C16, C17, C18, C19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
