File: hardware/SKnob.sch (KiCad schematic (older format))
At the start: 70 parts, among them J1 USB_B_Micro, J2 Conn_01x02, J3 Conn_01x02, Q1 FDV301N, SW1 SW_Push, T1 LA_LOGO, T2 LA_LOGO, U1 STM32WB55Cx, U2 LIS2DE12TR, U3 USBLC6-2P6, Y1 32MHz, Y2 32.768kHz

Commit message: hardware Rev 1.0
Parts:
- C17, C19: value 15pF -> 9pF
- J1: digikey# (none) -> WM9734CT-ND; info (none) -> USB - micro B USB 2.0 Receptacle Connector 5 Position Surfa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; manf (none) -> Molex; manf# (none) -> 1051330001
- J2, J3: digikey# (none) -> 952-2280-ND; info (none) -> Connector Header Through Hole 2 position 0.079\" (2.00mm); manf (none) -> Harwin Inc.; manf# (none) -> M22-2510246
- L1, L2: value 600R @ 100MHz -> 220 @ 100MHz; digikey# (none) -> 445-172893-1-ND; info (none) -> 220 Ohms @ 100MHz 1 Power Line Ferrite Bead 0603 (1608 Metr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; manf (none) -> TDK Corporation; manf# (none) -> 445-172893-1-ND
- Q1: info (none) -> N-Channel 25V 220mA (Ta) 350mW (Ta) Surface Mount SOT-23
- SW1: digikey# (none) -> SW1022CT-ND; info (none) -> SWITCH TACTILE SPST-NO 0.05A 12V; manf (none) -> Omron Electronics Inc-EMC Div; manf# (none) -> B3U-3000P
- Y2: footprint Crystal:Crystal_SMD_2016-4Pin_2.0x1.6mm -> Crystal:Crystal_SMD_2012-2Pin_2.0x1.2mm; symbol Device:Crystal_GND24 -> Device:Crystal; digikey# (none) -> XC2744CT-ND; info (none) -> 32.768kHz ±10ppm Crystal 9pF 70 kOhms 2-SMD, No Lead; manf (none) -> ECS Inc.; manf# (none) -> ECS-.327-9-12R-C-TR
- renumbered BATT?1 to BATT1
Connections:
- net GND: no longer Y2.2, Y2.4
- net OSC32_OUT: now also Y2.2; no longer Y2.3

Commit message: shopping carts from digikey and mouser, added mouser part numbers to sch
Parts:
- ANT1: mouser# (none) -> 673-W3008
- FLT1: mouser# (none) -> 511-MLPF-WB55-01E3
- J1: mouser# (none) -> 538-105133-0001
- J2, J3: mouser# (none) -> 855-M22-2510246
- L1, L2: mouser# (none) -> 810-MPZ1608S221ATD25
- L4: mouser# (none) -> 963-CBMF1608T100K
- Q1: mouser# (none) -> 512-FDV301N
- U1: mouser# (none) -> 511-STM32WB55CGU6
- U2: mouser# (none) -> 511-LIS2DE12TR
- U3: mouser# (none) -> 511-STEVAL-IPE023V1
- Y1: mouser# (none) -> 81-XRCGB32M000F1H02R
- Y2: mouser# (none) -> 520-.327-9-12R-C-T
Changed lines of the file:
@@
 F 6 "PulseLarsen Antennas" H 11550 6350 50  0001 C CNN "manf"
 F 7 "2.4GHz Bluetooth Chip RF Antenna 2.4GHz ~ 2.483GHz 1.7dBi Solder Surface Mount" H 11550 6350 50  0001 C CNN "info"
+F 8 "673-W3008" H 11550 6350 50  0001 C CNN "mouser#"
 	1    11550 6350
 	1    0    0    -1
@@
 F 6 "TDK Corporation" H 9050 2100 50  0001 C CNN "manf"
 F 7 "445-172893-1-ND" H 9050 2100 50  0001 C CNN "manf#"
+F 8 "810-MPZ1608S221ATD25" H 9050 2100 50  0001 C CNN "mouser#"
 	1    9050 2100
 	0    -1   -1   0
@@
 F 6 "WM9734CT-ND" H 1700 4100 50  0001 C CNN "digikey#"
 F 7 "USB - micro B USB 2.0 Receptacle Connector 5 Position Surface Mount" H 1700 4100 50  0001 C CNN "info"
+F 8 "538-105133-0001" H 1700 4100 50  0001 C CNN "mouser#"
 	1    1700 4100
 	1    0    0    -1
@@
 F 6 "STM32WB55CGU6" H 6400 4750 50  0001 C CNN "manf#"
 F 7 "IC RF TxRx + MCU 802.15.4, Bluetooth Bluetooth v5.0 2.405GHz ~ 2.48GHz 48-UFQFN Exposed Pad" H 6400 4750 50  0001 C CNN "info"
+F 8 "511-STM32WB55CGU6" H 6400 4750 50  0001 C CNN "mouser#"
 	1    6400 4750
 	1    0    0    -1
@@
 F 6 "TDK Corporation" H 9050 2850 50  0001 C CNN "manf"
 F 7 "445-172893-1-ND" H 9050 2850 50  0001 C CNN "manf#"
+F 8 "810-MPZ1608S221ATD25" H 9050 2850 50  0001 C CNN "mouser#"
 	1    9050 2850
 	0    -1   -1   0
@@
 F 6 "587-1720-1-ND" V 8750 3900 50  0001 C CNN "digikey#"
 F 7 "10µH Unshielded Wirewound Inductor 380mA 468mOhm Max 0603 (1608 Metric)" H 8750 3900 50  0001 C CNN "info"
+F 8 "963-CBMF1608T100K" H 8750 3900 50  0001 C CNN "mouser#"
 	1    8750 3900
 	0    -1   -1   0
@@
 F 6 "XRCGB32M000F1H02R0" H 14450 4550 50  0001 C CNN "manf#"
 F 7 "32MHz ±10ppm Crystal 10pF 60 Ohms 4-SMD, No Lead" H 14450 4550 50  0001 C CNN "info"
+F 8 " 81-XRCGB32M000F1H02R " H 14450 4550 50  0001 C CNN "mouser#"
 	1    14450 4550
 	1    0    0    -1
@@
 F 6 "ECS Inc." H 14450 6200 50  0001 C CNN "manf"
 F 7 "ECS-.327-9-12R-C-TR" H 14450 6200 50  0001 C CNN "manf#"
+F 8 " 520-.327-9-12R-C-T " H 14450 6200 50  0001 C CNN "mouser#"
 	1    14450 6200
 	1    0    0    -1
@@
 F 6 "Harwin Inc." H 2850 1500 50  0001 C CNN "manf"
 F 7 "M22-2510246" H 2850 1500 50  0001 C CNN "manf#"
+F 8 "855-M22-2510246" H 2850 1500 50  0001 C CNN "mouser#"
 	1    2850 1500
 	1    0    0    -1
@@
 F 6 "Harwin Inc." H 12100 8450 50  0001 C CNN "manf"
 F 7 "M22-2510246" H 12100 8450 50  0001 C CNN "manf#"
+F 8 "855-M22-2510246" H 12100 8450 50  0001 C CNN "mouser#"
 	1    12100 8450
 	-1   0    0    -1
@@
 F 6 "497-15997-1-ND " H 2250 9700 50  0001 C CNN "digikey#"
 F 7 "Accelerometer X, Y, Z Axis ±2g, 4g, 8g, 16g 0.5Hz ~ 2.69kHz 12-LGA (2x2)" H 2250 9700 50  0001 C CNN "info"
+F 8 "511-LIS2DE12TR " H 2250 9700 50  0001 C CNN "mouser#"
 	1    2250 9700
 	1    0    0    -1
@@
 F 6 "USBLC6-2P6" H 2200 6350 50  0001 C CNN "manf#"
 F 7 "17V Clamp 5A (8/20µs) Ipp Tvs Diode Surface Mount SOT-666" H 2200 6350 50  0001 C CNN "info"
+F 8 "511-STEVAL-IPE023V1" H 2200 6350 50  0001 C CNN "mouser#"
 	1    2200 6350
 	1    0    0    -1
@@
 F 6 "MLPF-WB55-01E3" H 10650 6450 50  0001 C CNN "manf#"
 F 7 "2.45GHz Center Frequency Low Pass RF Filter (Radio Frequency) 100MHz Bandwidth 1.1dB 6-SMD, No Lead" H 10650 6450 50  0001 C CNN "info"
+F 8 "511-MLPF-WB55-01E3 " H 10650 6450 50  0001 C CNN "mouser#"
 	1    10650 6450
 	1    0    0    -1
@@
 F 6 "FDV301NCT-ND" H 10650 10700 50  0001 C CNN "digikey#"
 F 7 "N-Channel 25V 220mA (Ta) 350mW (Ta) Surface Mount SOT-23" H 10650 10700 50  0001 C CNN "info"
+F 8 "512-FDV301N " H 10650 10700 50  0001 C CNN "mouser#"
 	1    10650 10700
 	1    0    0    -1
