File: hardware/SKnob.kicad_pcb (KiCad board)
At the start: 4 copper layers, 50 x 17 mm, 71 parts, among them J1 USB_B_Micro, J2 Conn_01x02, J3 Conn_01x02, Q1 FDV301N, SW1 SW_Push, T1 LA_LOGO, T2 LA_LOGO, U1 STM32WB55Cx, U2 LIS2DE12TR, U3 USBLC6-2P6, Y1 32MHz, Y2 32.768kHz

Commit message: remove silk from footprints, replace silk gerber with empty manually
Routing:
- net /RF1_ANT: track 7.61 -> 7.10 mm
- net (no net): vias 0 -> 8
Other:
- outline, holes or cut-outs redrawn
- net class microstrip: trace_width 0.29337 -> 0.25
- net class usb: trace_width 0.118 -> 0.2
- board text added: "Top Layer 50 Ohm microstrip"
- board text added: "Top Layer 90 Ohm differential microstrip"
- board text added: "Top Paste Top Soldermask 1 - Top Copper (35 um Final) Prepreg 2x ISOLA IS400 (125 um Final) 2 - Inner Copper (35 um) Core (1200 um) 3 - Inner Copper (35 um) Prepreg 2x ISOLA IS400 (125 um Final) 4 - Bottom Copper (35 um Final) Bottom Soldermask Total thickness: 1.6 mm"
